File: UAV_FC.kicad_sch (KiCad schematic)
At the start: 0 parts

Commit message: 4/8 Progress
Parts:
- added C1, C13, C15, C16, C18, C2, C21, C22, C24, C3, C32, C33, C34, C35, C36, C4, C5, C6, C7, C8, C9: 100n, Capacitor_SMD:C_0402_1005Metric, symbol Device:C
- added C10, C11, C12, C14, C23: 4.7u, Capacitor_SMD:C_0402_1005Metric, symbol Device:C
- added C17, C37, C38: 10u, Capacitor_SMD:C_0402_1005Metric, symbol Device:C
- added C19, C20: 15p, Capacitor_SMD:C_0402_1005Metric, symbol Device:C
- added C25, C26: 10u, Capacitor_SMD:C_0805_2012Metric, symbol Device:C
- added C27: 10n, Capacitor_SMD:C_0402_1005Metric, symbol Device:C
- added C28, C29: 100u, Capacitor_SMD:C_1206_3216Metric, symbol Device:C
- added D1: WHITE, Diode_SMD:D_0603_1608Metric, symbol Device:LED
- added D2, D3: RED, Diode_SMD:D_0603_1608Metric, symbol Device:LED
- added D4: 550mV/40V, Diode_SMD:D_SMA, symbol Device:D_Schottky
- added FID1, FID2, FID3: Fiducial, Fiducial:Fiducial_1mm_Mask2mm, symbol Mechanical:Fiducial
- added H1, H2, H3, H4: MountingHole, MountingHole:MountingHole_4.3mm_M4, symbol Mechanical:MountingHole
- added J1: USB_C_Receptacle_USB2.0_16P, Connector_USB:USB_C_Receptacle_HRO_TYPE-C-31-M-12, symbol Connector:USB_C_Receptacle_USB2.0_16P
- added J2: JST Debug Connector, Connector_JST:JST_SH_BM03B-SRSS-TB_1x03-1MP_P1.00mm_Vertical, symbol Connector_Generic_MountingPin:Conn_01x03_MountingPin
- added J3: GPS Connector, Connector_JST:JST_SH_SM06B-SRSS-TB_1x06-1MP_P1.00mm_Horizontal, symbol Connector_Generic_MountingPin:Conn_01x06_MountingPin
- added J4: 4-in1 ESC Connector, Connector_JST:JST_SH_SM08B-SRSS-TB_1x08-1MP_P1.00mm_Horizontal, symbol Connector_Generic_MountingPin:Conn_01x08_MountingPin
- added J5: ELRS Receiver Connector, Connector_JST:JST_SH_SM04B-SRSS-TB_1x04-1MP_P1.00mm_Horizontal, symbol Connector_Generic_MountingPin:Conn_01x04_MountingPin
- added L1: 3.3u, Inductor_SMD:AOTA-B201610S3R3-101-T, symbol Device:L
- added L2: 33u, Inductor_SMD:L_Cenker_CKCS8060, symbol Device:L
- added R1, R2: 27, Resistor_SMD:R_0402_1005Metric, symbol Device:R
- added R10, R16, R17, R8: 10k, Resistor_SMD:R_0402_1005Metric, symbol Device:R
- added R11, R12, R13, R14, R7, R9: 1k, Resistor_SMD:R_0402_1005Metric, symbol Device:R
- added R15: 100k, Resistor_SMD:R_0402_1005Metric, symbol Device:R
- added R18: 3.24k, Resistor_SMD:R_0402_1005Metric, symbol Device:R
- added R19, R20, R23, R24: 4.7k, Resistor_SMD:R_0402_1005Metric, symbol Device:R
- added R3: 33, Resistor_SMD:R_0402_1005Metric, symbol Device:R
- added R4: 600/100, Resistor_SMD:R_0805_2012Metric, symbol Device:R
- added R5, R6: 5.1k, Resistor_SMD:R_0402_1005Metric, symbol Device:R
- added SW1, SW2: SW_Push, Button_Switch_SMD:SW_SPST_TS-1088-xR020, symbol Switch:SW_Push
- added U1: RP2350_80QFN, RP2350_80QFN_minimal:RP2350-QFN-80-1EP_10x10_P0.4mm_EP3.4x3.4mm_ThermalVias, symbol MCU_RaspberryPi_RP2350:RP2350_80QFN
- added U2: USBLC6-2SC6, Package_TO_SOT_SMD:SOT-23-6, symbol Power_Protection:USBLC6-2SC6
- added U3: W25Q128JVS, Package_SO:SOIC-8_5.3x5.3mm_P1.27mm, symbol Memory_Flash:W25Q128JVS
- added U5: TPS5430DDA, Package_SO:TI_SO-PowerPAD-8_ThermalVias, symbol Regulator_Switching:TPS5430DDA
- added U6: BMI088, Package_LGA:Bosch_LGA-16_4.5x3mm_P0.5mm_LayoutBorder7x1y_ClockwisePinNumbering, symbol Sensor_Motion:BMI088
- added U7: ICM-45686, Package_LGA:LGA-14_3x2.5mm_P0.5mm_LayoutBorder3x4y, symbol Drone:ICM-45686
- added U8: LPS22HH, Package_LGA:ST_HLGA-10_2x2mm_P0.5mm_LayoutBorder3x2y, symbol Sensor_Pressure:LPS22HH
- added U9: SPX3819M5-L-3-3, Package_TO_SOT_SMD:SOT-23-5, symbol Regulator_Linear:SPX3819M5-L-3-3
- added Y1: ABM8-272-T3, Crystal:Crystal_SMD_Abracon_ABM8AIG-4Pin_3.2x2.5mm, symbol Device:Crystal_GND24
Connections:
- new net: D1.1 (K), R14.2
- new net: C36.1, U9.4 (BP)
- new net: D3.1 (K), R13.2
- new net: R2.1, U1.66 (USB_DM)
- new net: R1.1, U1.67 (USB_DP)
- new net: C27.2, D4.1 (K), L2.1, U5.8 (PH)
- new net: D2.1 (K), R12.2
- new net: R11.2, SW1.1
- new net: R17.1, R18.2, U5.4 (VSENSE)
- new net: J1.A7 (D-), J1.B7 (D-), U2.1 (I/O1)
- new net: J1.A6 (D+), J1.B6 (D+), U2.3 (I/O2)
- new net: C20.2, R9.1, Y1.3
- new net: C27.1, U5.1 (BOOT)
- new net: R7.1, SW2.2
- new net +1V1: C10.1, C13.1, C14.1, C15.1, L1.1, U1.10 (DVDD), U1.32 (DVDD), U1.51 (DVDD), U1.65 (VREG_FB)
- new net +3V3: C1.1, C11.1, C18.1, C2.1, C22.1, C23.1, C3.1, C32.1, C33.1, C34.1, C35.1, C37.1, C4.1, C5.1, C6.1, C7.1, C8.1, C9.1, D2.2 (A), R10.2, R19.1, R20.1, R23.1, R24.1, R3.2, R8.1, U1.15 (IOVDD), U1.24 (IOVDD), U1.29 (IOVDD), U1.41 (IOVDD), U1.5 (IOVDD), U1.50 (IOVDD), U1.59 (ADC_AVDD), U1.60 (IOVDD), U1.64 (VREG_VIN), U1.68 (USB_OTP_VDD), U1.69 (QSPI_IOVDD), U1.76 (IOVDD), U3.8 (VCC), U6.11 (VDDIO), U6.3 (VDD), U7.5 (VDDIO), U7.8 (VDD), U8.1 (Vdd_IO), U8.10 (VDD), U8.5 (SA0), U8.6 (~{CS}), U9.5 (OUT)
- new net +5V: C17.1, C28.1, C29.1, C38.1, D3.2 (A), J3.5 (Pin_5), J5.2 (Pin_2), L2.2, R17.2, R4.1, U9.1 (IN), U9.3 (EN)
- new net +VBUS: C16.1, J1.A4 (VBUS), J1.A9 (VBUS), J1.B4 (VBUS), J1.B9 (VBUS), R4.2, U2.5 (VBUS)
- new net BMTR_INT: U8.7 (INT_DRDY)
- new net BMTR_SCL: R24.2, U1.80 (GPIO3), U8.2 (SCL)
- new net BMTR_SDA: R23.2, U1.79 (GPIO2), U8.4 (SDA)
- new net C: J4.7 (Pin_7), U1.49 (GPIO40_ADC0)
- new net CMPS_SCL: J3.1 (Pin_1), R19.2, U1.37 (GPIO29)
- new net CMPS_SDA: J3.2 (Pin_2), R20.2, U1.38 (GPIO30)
- new net ELRS_RX: J5.4 (Pin_4), U1.1 (GPIO4)
- new net ELRS_TX: J5.3 (Pin_3), U1.2 (GPIO5)
- new net FLASH_CLK: U1.71 (QSPI_SCLK), U3.6 (CLK)
- new net FLASH_CS: R7.2, R8.2, U1.75 (QSPI_SS), U3.1 (~{CS})
- new net FLASH_IO0: U1.72 (QSPI_SD0), U3.5 (DI/IO_{0})
- new net FLASH_IO1: U1.74 (QSPI_SD1), U3.2 (DO/IO_{1})
- new net FLASH_IO2: U1.73 (QSPI_SD2), U3.3 (~{WP}/IO_{2})
- new net FLASH_IO3: U1.70 (QSPI_SD3), U3.7 (~{HOLD}/~{RESET}/IO_{3})
- new net GND: C1.2, C10.2, C11.2, C12.2, C13.2, C14.2, C15.2, C16.2, C17.2, C18.2, C19.1, C2.2, C20.1, C21.2, C22.2, C23.2, C24.2, C25.2, C26.2, C28.2, C29.2, C3.2, C32.2, C33.2, C34.2, C35.2, C36.2, C37.2, C38.2, C4.2, C5.2, C6.2, C7.2, C8.2, C9.2, D4.2 (A), J1.A1 (GND), J1.A12 (GND), J1.B1 (GND), J1.B12 (GND), J1.S1 (SHIELD), J2.2 (Pin_2), J2.MP (MountPin), J3.6 (Pin_6), J3.MP (MountPin), J4.1 (Pin_1), J4.MP (MountPin), J5.1 (Pin_1), J5.MP (MountPin), R11.1, R12.1, R13.1, R14.1, R16.1, R18.1, R5.2, R6.2, SW2.1, U1.62 (VREG_PGND), U1.81 (GND), U2.2 (GND), U3.4 (GND), U5.6 (GND), U5.9 (GNDPAD), U6.2 (GNDA), U6.4 (GNDA), U6.6 (GNDIO), U6.7 (PS), U7.6 (GND), U8.3 (GND), U8.8 (GND), U8.9 (GND), U9.2 (GND), Y1.2, Y1.4
- new net GPS_RX: J3.3 (Pin_3), U1.39 (GPIO31)
- new net GPS_TX: J3.4 (Pin_4), U1.40 (GPIO32)
- new net IMU2_CS1: U1.9 (GPIO11), U6.14 (~{CSB1})
- new net IMU2_CS2: U1.12 (GPIO13), U6.5 (~{CSB2})
- new net IMU2_INT1: U1.8 (GPIO10), U6.16 (INT1)
- new net IMU2_INT3: U1.18 (GPIO18), U6.12 (INT3)
- new net IMU2_SCLK: U1.13 (GPIO14), U6.8 (SCK/SCL)
- new net IMU2_SDI: U1.14 (GPIO15), U6.9 (SDI/SDA)
- new net IMU2_SDO: U1.11 (GPIO12), U6.10 (SDO2), U6.15 (SDO1)
- new net IMU_CS: U1.21 (GPIO21), U7.12 (AP_CS)
- new net IMU_INT: U1.19 (GPIO19), U7.4 (INT1/INT)
- new net IMU_SCLK: U1.22 (GPIO22), U7.13 (AP_SCLK)
- new net IMU_SDI: U1.23 (GPIO23), U7.14 (AP_SDIO/AP_SDI)
- new net IMU_SDO: U1.20 (GPIO20), U7.1 (AP_SDO)
- new net M1: J4.3 (Pin_3), U1.45 (GPIO36)
- new net M2: J4.4 (Pin_4), U1.46 (GPIO37)
- new net M3: J4.5 (Pin_5), U1.47 (GPIO38)
- new net M4: J4.6 (Pin_6), U1.48 (GPIO39)
- new net RUN: R10.1, SW1.2, U1.35 (RUN)
- new net STATUS: D1.2 (A), U1.53 (GPIO42_ADC2)
- new net SWCLK: J2.1 (Pin_1), U1.33 (SWCLK)
- new net SWD: J2.3 (Pin_3), U1.34 (SWD)
- new net USBCC1: J1.A5 (CC1), R6.1
- new net USBCC2: J1.B5 (CC2), R5.1
- new net USBD+: R1.2, U2.4 (I/O2)
- new net USBD-: R2.2, U2.6 (I/O1)
- new net VBAT: C24.1, C25.1, C26.1, J4.2 (Pin_2), R15.2, U5.7 (VIN)
- new net VBAT_ADC: C21.1, R15.1, R16.2, U1.52 (GPIO41_ADC1)
- new net VREG_AVDD: C12.1, R3.1, U1.61 (VREG_AVDD)
- new net VREG_LX: L1.2, U1.63 (VREG_LX)
- new net XIN: C19.2, U1.30 (XIN), Y1.1
- new net XOUT: R9.2, U1.31 (XOUT)
- no-connect marks 0 -> 33
Other:
- note added: "CRYSTAL"
- note added: "DEBUG/STATUS"
- note added: "GPS/ESC/RF CONNECTORS"
- note added: "MCU + CORE REGULATOR CIRCUIT"
- note added: "PERIPHERAL"
- note added: "POWER"
- note added: "QSPI FLASH"
- note added: "USB CONNECTOR"

Commit message: 4/26 update
Parts:
- removed C15, C36: 100n, Capacitor_SMD:C_0402_1005Metric, symbol Device:C
- removed L1: 3.3u, Inductor_SMD:AOTA-B201610S3R3-101-T, symbol Device:L
- removed R2: 27, Resistor_SMD:R_0402_1005Metric, symbol Device:R
- removed R3: 33, Resistor_SMD:R_0402_1005Metric, symbol Device:R
- removed U1: RP2350_80QFN, RP2350_80QFN_minimal:RP2350-QFN-80-1EP_10x10_P0.4mm_EP3.4x3.4mm_ThermalVias, symbol MCU_RaspberryPi_RP2350:RP2350_80QFN
- removed U9: SPX3819M5-L-3-3, Package_TO_SOT_SMD:SOT-23-5, symbol Regulator_Linear:SPX3819M5-L-3-3
- added FB1: 600Ω@100MHz, Inductor_SMD:L_0603_1608Metric, symbol Device:FerriteBead
- added SW3, SW4: SW_Push, Button_Switch_SMD:SW_SPST_TS-1088-xR020, symbol Switch:SW_Push
- added U1: STM32H743VITx, Package_QFP:LQFP-100_14x14mm_P0.5mm, symbol MCU_ST_STM32H7:STM32H743VITx
- added U4: TLV75733PDBV, Package_TO_SOT_SMD:SOT-23-5, symbol Regulator_Linear:TLV75733PDBV
- C1: value 100n -> 4.7u; Distributor Link 1 https://www.mouser.com/ProductDetail/Samsung-Electro-Mechan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 -> https://www.digikey.com/en/products/detail/samsung-electro-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; Distributor Link 2 https://www.digikey.com/en/products/detail/samsung-electro-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 -> https://www.mouser.com/ProductDetail/Samsung-Electro-Mechan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; LCSC C1525 -> C23733; Manufacturer Part Number CL05B104KO5NNNC -> CL05A475MP5NRNC
- C10, C14: value 4.7u -> 100n; Distributor Link 1 https://www.digikey.com/en/products/detail/samsung-electro-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 -> https://www.mouser.com/ProductDetail/Samsung-Electro-Mechan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; Distributor Link 2 https://www.mouser.com/ProductDetail/Samsung-Electro-Mechan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 -> https://www.digikey.com/en/products/detail/samsung-electro-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; LCSC C23733 -> C1525; Manufacturer Part Number CL05A475MP5NRNC -> CL05B104KO5NNNC
- C11: value 4.7u -> 1u; Distributor Link 1 https://www.digikey.com/en/products/detail/samsung-electro-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 -> https://www.mouser.com/ProductDetail/Samsung-Electro-Mechan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; Distributor Link 2 https://www.mouser.com/ProductDetail/Samsung-Electro-Mechan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 -> https://www.digikey.com/en/products/detail/samsung-electro-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; LCSC C23733 -> C52923; Manufacturer Part Number CL05A475MP5NRNC -> CL05A105KA5NQNC
- C12: value 4.7u -> 2.2u; Distributor Link 1 https://www.digikey.com/en/products/detail/samsung-electro-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 -> https://www.mouser.com/ProductDetail/Samsung-Electro-Mechan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; Distributor Link 2 https://www.mouser.com/ProductDetail/Samsung-Electro-Mechan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 -> https://www.digikey.com/en/products/detail/samsung-electro-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; LCSC C23733 -> C12530; Manufacturer Part Number CL05A475MP5NRNC -> CL05A225MQ5NSNC
- C13: value 100n -> 2.2u; Distributor Link 1 https://www.mouser.com/ProductDetail/Samsung-Electro-Mechanics/CL05B104KO5NNNC?qs=hqM3L16%252BxlfT2SKOuAUq6Q%3D%3D -> https://www.mouser.com/ProductDetail/Samsung-Electro-Mechanics/CL05A225MQ5NSNC?qs=X6jEic%2FHinC0eBcvtpjFyQ%3D%3D; Distributor Link 2 https://www.digikey.com/en/products/detail/samsung-electro-mechanics/CL05B104KO5NNNC/3886659?s=N4IgTCBcDaIMIBkAMBWAQgRiQFgNIHkUA5EuEAXQF8g -> https://www.digikey.com/en/products/detail/samsung-electro-mechanics/CL05A225MQ5NSNC/3887129?s=N4IgTCBcDaIMIBkAMBWAgmMKCyBFFAcgMoFwgC6AvkA; LCSC C1525 -> C12530; Manufacturer Part Number CL05B104KO5NNNC -> CL05A225MQ5NSNC
- C9: value 100n -> 1u; Distributor Link 1 https://www.mouser.com/ProductDetail/Samsung-Electro-Mechanics/CL05B104KO5NNNC?qs=hqM3L16%252BxlfT2SKOuAUq6Q%3D%3D -> https://www.mouser.com/ProductDetail/Samsung-Electro-Mechanics/CL05A105KA5NQNC?qs=X6jEic%2FHinDIeFgZnm60Lw%3D%3D; Distributor Link 2 https://www.digikey.com/en/products/detail/samsung-electro-mechanics/CL05B104KO5NNNC/3886659?s=N4IgTCBcDaIMIBkAMBWAQgRiQFgNIHkUA5EuEAXQF8g -> https://www.digikey.com/en/products/detail/samsung-electro-mechanics/CL05A105KA5NQNC/3887103?s=N4IgTCBcDaIMIBkAMBWAggRlQaTSgcgIr5wgC6AvkA; LCSC C1525 -> C52923; Manufacturer Part Number CL05B104KO5NNNC -> CL05A105KA5NQNC
- R1: value 27 -> 10k; LCSC C25100 -> C25744; Manufacturer Part Number 0402WGF270JTCE -> 0402WGF1002TCE
Connections:
- net +3V3: now also FB1.2, SW4.1, U1.100 (VDD), U1.11 (VDD), U1.27 (VDD), U1.50 (VDD), U1.6 (VBAT), U1.75 (VDD), U4.5 (OUT); no longer C11.1, C8.1, C9.1
- net +5V: now also U4.1 (IN), U4.3 (EN)
- net GND: now also R1.2, SW3.1, U1.10 (VSS), U1.19 (VSSA), U1.26 (VSS), U1.49 (VSS), U1.74 (VSS), U1.99 (VSS), U4.2 (GND)
- net USBD+: no longer R1.2
- net at R1.1: now also SW4.2, U1.94 (BOOT0)
- removed net +1V1: C10.1, C13.1, C14.1
- net VREG_AVDD: no longer names the net of C12.1
- net VREG_AVDD: now also C13.1, U1.48 (VCAP), U1.73 (VCAP)
- new net: C14.1, SW3.2, U1.14 (NRST)
- new net VDDA: C10.1, C11.1, C8.1, C9.1, FB1.1, U1.20 (VREF+), U1.21 (VDDA)
- no-connect marks 33 -> 12
Other:
- note removed: "MCU + CORE REGULATOR CIRCUIT"
- moved on the sheet: C37, C38

Commit message: May 6th
Parts:
- added J6: Micro_SD_Card_Det_Hirose_DM3AT, Connector_Card:microSD_HC_Hirose_DM3AT-SF-PEJM5, symbol Connector:Micro_SD_Card_Det_Hirose_DM3AT
- added J7: DroneCAN Connector, Connector_JST:JST_GH_SM04B-GHS-TB_1x04-1MP_P1.25mm_Horizontal, symbol Connector_Generic_MountingPin:Conn_01x04_MountingPin
- added J8: MAVLink Connector, Connector_JST:JST_GH_SM05B-GHS-TB_1x05-1MP_P1.25mm_Horizontal, symbol Connector_Generic_MountingPin:Conn_01x05_MountingPin
- added R2, R21, R22, R25, R3: 10k, Resistor_SMD:R_0402_1005Metric, symbol Device:R
- added R26: 120, Resistor_SMD:R_0402_1005Metric, symbol Device:R
- added U9: TJA1051TK-3, Package_SON:HVSON-8-1EP_3x3mm_P0.65mm_EP1.6x2.4mm, symbol Interface_CAN_LIN:TJA1051TK-3
Connections:
- net +3V3: now also J6.4 (VDD), R2.2, R21.2, R22.2, R25.2, R3.2, U9.5 (VIO)
- net +5V: now also J7.1 (Pin_1), U9.3 (VCC)
- net BMTR_SCL: now also U1.92 (PB6)
- net BMTR_SDA: now also U1.93 (PB7)
- net FLASH_CLK: now also U1.36 (PB2)
- net FLASH_CS: now also U1.79 (PC11)
- net FLASH_IO0: now also U1.37 (PE7)
- net FLASH_IO1: now also U1.38 (PE8)
- net FLASH_IO2: now also U1.39 (PE9)
- net FLASH_IO3: now also U1.40 (PE10)
- net GND: now also J6.11 (SHIELD), J6.6 (VSS), J6.9 (DET_B), J7.4 (Pin_4), J7.MP (MountPin), J8.1 (Pin_1), J8.MP (MountPin), U9.2 (GND), U9.8 (S), U9.9 (GND)
- net IMU2_SCLK: now also U1.52 (PB13)
- net IMU2_SDI: now also U1.54 (PB15)
- net IMU2_SDO: now also U1.53 (PB14)
- net IMU_SCLK: now also U1.42 (PE12)
- net IMU_SDI: now also U1.44 (PE14)
- net IMU_SDO: now also U1.43 (PE13)
- net USBD+: now also U1.71 (PA12)
- net USBD-: now also U1.70 (PA11)
- net XIN: now also U1.12 (PH0)
- net XOUT: now also U1.13 (PH1)
- net ESC_TLM: now reaches J4.8 (Pin_8)
- net SD_DATA: now reaches U1.65 (PC8)
- net SD_DATA: now also J6.7 (DAT0), R22.1
- net SD_CLK: now reaches U1.80 (PC12)
- net SD_CLK: now also J6.5 (CLK)
- net SD_CMD: now reaches U1.83 (PD2)
- net SD_CMD: now also J6.3 (CMD), R21.1
- net CAN_RX: now reaches U1.95 (PB8)
- net CAN_RX: now also U9.4 (RXD)
- net CAN_TX: now reaches U1.96 (PB9)
- net CAN_TX: now also U9.1 (TXD)
- net C renamed ESC_CURR
- new net: J6.1 (DAT2), R2.1
- new net: J6.2 (DAT3/CD), R3.1
- new net: J6.8 (DAT1), R25.1
- new net: J7.2 (Pin_2), R26.1, U9.7 (CANH)
- new net: J7.3 (Pin_3), R26.2, U9.6 (CANL)
- new net SD_DET: J6.10 (DET_A)
- new net USART_CTS: J8.5 (Pin_5)
- new net USART_RTS: J8.4 (Pin_4)
- new net USART_RX: J8.3 (Pin_3)
- new net USART_TX: J8.2 (Pin_2)
- no-connect marks 12 -> 11
Other:
- moved on the sheet: C1, C10, C11, C12, C13, C14, C16, C17, C18, C19, C2, C20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
